Commit message: recorded primarily demo video

File: fastpick_description/xacro/franka_arm.urdf.xacro (robot description, xacro)
@@ -11,8 +11,8 @@
     <!-- Create a URDF for a real hardware -->
     <xacro:include filename="$(find franka_description)/robots/panda_arm.xacro" />
-    <xacro:panda_arm arm_id="$(arg arm_id)" safety_distance="0.03"/>
+    <xacro:panda_arm arm_id="$(arg arm_id)" safety_distance="0.0"/>
     <xacro:if value="$(arg hand)">
       <xacro:include filename="$(find franka_description)/robots/hand.xacro"/>
-      <xacro:hand arm_id="$(arg arm_id)" rpy="0 0 ${-pi/4}" xyz="0 0 0.005" connected_to="$(arg arm_id)_link8" safety_distance="0.03"/>
+      <xacro:hand arm_id="$(arg arm_id)" rpy="0 0 ${-pi/4}" xyz="0 0 0.005" connected_to="$(arg arm_id)_link8" safety_distance="0.0"/>
     </xacro:if>
   </xacro:unless>

File: panda_moveit_config/config/panda_arm.xacro (robot description, xacro)
@@ -48,4 +48,14 @@
       <joint name="panda_joint7" value="0.7457435544252466" />
     </group_state>
+<!-- [0.05314294423578273 -0.9757922195425274 -0.10976040384865092 -2.764346203988058 0.02037217205167416 3.016741504351298 0.6674461618982057] -->
+    <group_state name="pick_start" group="panda_arm">
+      <joint name="panda_joint1" value="0.05314294423578273" />
+      <joint name="panda_joint2" value="-0.9757922195425274" />
+      <joint name="panda_joint3" value="-0.10976040384865092" />
+      <joint name="panda_joint4" value="-2.764346203988058" />
+      <joint name="panda_joint5" value="0.02037217205167416" />
+      <joint name="panda_joint6" value="3.016741504351298" />
+      <joint name="panda_joint7" value="0.6674461618982057" />
+    </group_state>
     <!--END EFFECTOR: Purpose: Represent information about an end effector.-->
     <!--VIRTUAL JOINT: Purpose: this element defines a virtual joint between a robot link and an external frame of reference (considered fixed with respect to the robot)-->
