Commit message: picking is working, work on octomap

File: panda_moveit_config/config/panda_arm.xacro (robot description, xacro)
@@ -58,4 +58,14 @@
       <joint name="panda_joint7" value="0.6674461618982057" />
     </group_state>
+<!-- [0.0703047732482682 0.11600033845239728 -0.13870497079407706 -2.478550928115845 0.03154783239938 2.6181519791285197 0.6776919333220165] -->
+    <group_state name="place_start" group="panda_arm">
+      <joint name="panda_joint1" value="0.0703047732482682" />
+      <joint name="panda_joint2" value="0.11600033845239728" />
+      <joint name="panda_joint3" value="-0.13870497079407706" />
+      <joint name="panda_joint4" value="-2.478550928115845" />
+      <joint name="panda_joint5" value="0.03154783239938" />
+      <joint name="panda_joint6" value="2.6181519791285197" />
+      <joint name="panda_joint7" value="0.6776919333220165" />
+    </group_state>
     <!--END EFFECTOR: Purpose: Represent information about an end effector.-->
     <!--VIRTUAL JOINT: Purpose: this element defines a virtual joint between a robot link and an external frame of reference (considered fixed with respect to the robot)-->
